File: hardware/nrf54.kicad_pcb (KiCad board)
At the start: 4 copper layers, 21 x 91 mm, 102 parts, among them J1 USB_C_Receptacle_USB2.0_14P, J10 U.FL, J2 Conn_01x10, J3 Conn_01x10, J4 Conn_01x03, J5 Conn_01x20, J6 Conn_01x20, J7 Conn_01x03, J8 USB_C_Receptacle_USB2.0_14P, J9 U.FL, Q2 RUM001L02, SW1 SW_Push, SW2 SW_Push, U1 NRF54L15-QFAA-R, U2 NPM1300-QEAA-R, U3 nRF52820-QDxx, U4 TPS63900, Y1 32MHz, Y2 32MHz, Y3 32.768kHz

Commit message: Stash
Parts:
- removed H1: MountingHole, nrf54:Icy Electronics Logo
- added H2: MountingHole, nrf54:Icy Electronics Logo, B.Cu at (81.9, 112.0)
- added JP4: SolderJumper_2_Open, PCM_ckl-misc:SolderJumper-2_Open_Pad_Small, B.Cu at (85.5, 112.9)
- added SW3: SW_Push, nrf54:SW_Push_SPST_TSA016, F.Cu at (79.3, 115.5)
- J1, J8: footprint Connector_USB:USB_C_Receptacle_HRO_TYPE-C-31-M-12 -> PCM_ckl-connector:USB_C_Receptacle_HRO_TYPE-C-31-M-12
- J2, J3: footprint Connector_PinHeader_2.54mm:PinHeader_1x10_P2.54mm_Vertical -> nrf54:Castellated_1x10_P2.54mm_Vertical
- J5, J6: footprint Connector_PinHeader_2.54mm:PinHeader_1x20_P2.54mm_Vertical -> nrf54:Castellated_1x20_P2.54mm_Vertical
- R2: footprint Capacitor_SMD:C_0402_1005Metric -> Resistor_SMD:R_0402_1005Metric
- moved TP3 4.28 mm to (84.8, 107.8)
- moved TP9 2.60 mm to (87.0, 105.6)
- moved TP4 1.81 mm to (87.7, 111.5)
- moved TP7 1.50 mm to (80.9, 77.0)
- moved H2 1.34 mm to (87.7, 41.9)
- moved J6 0.98 mm to (93.9, 41.7)
- moved J2 0.97 mm to (74.1, 95.0)
- moved J3 0.97 mm to (93.9, 95.0)
- moved J5 0.97 mm to (74.1, 41.7)
- moved TP1 0.51 mm to (79.5, 104.3)
- moved TP8 0.29 mm to (80.2, 74.8)
- moved TP2 0.08 mm to (80.0, 102.3)
Routing:
- net /nrf52820/P0.06: track 16.4 -> 20.7 mm, vias 0 -> 2
- net GND: track 53.1 -> 51.2 mm, vias 140 -> 159
- net VDD: track 96.6 -> 97.4 mm
- net /nrf52820/TXD: track 90.0 -> 90.6 mm
- net /nrf52820/SEL: track 2.19 -> 2.20 mm, vias 0 -> 1
Other:
- board size 21 x 91 mm -> 21 x 91.2 mm
- board text removed: "TXD RXD SWCLK SWDIO"
