File: hardware/nrf54.kicad_sch (KiCad schematic)
At the start: 2 parts

Commit message: Stash
Parts:
- H3, H4: now not fitted
Changed lines of the file:
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@@
 		(on_board yes)
 		(in_pos_files yes)
-		(dnp no)
+		(dnp yes)
 		(fields_autoplaced yes)
 		(property "Reference" "H4"
@@
 		(on_board yes)
 		(in_pos_files yes)
-		(dnp no)
+		(dnp yes)
 		(fields_autoplaced yes)
 		(property "Reference" "H3"

Commit message: Add schematic
Other:
- title: (none) -> nRF54L15 Discovery
Changed lines of the file:
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@@
 	(paper "A4")
 	(title_block
+		(title "nRF54L15 Discovery")
+		(date "05/06/2026")
+		(rev "v1.0")
 		(company "Icy Electronics")
+		(comment 1 "Chengyin (cheyao)")
 	)
 	(wire
