File: hardware/nrf54l15.kicad_sch (KiCad schematic)
At the start: 55 parts, among them J5 Conn_01x20, J6 Conn_01x20, J7 Conn_01x03, J8 USB_C_Receptacle_USB2.0_14P, J9 U.FL, Q2 RUM001L02, SW1 SW_Push, SW2 SW_Push, U1 NRF54L15-QFAA-R, U2 NPM1300-QEAA-R, Y1 32MHz, Y3 32.768kHz

Commit message: Stash
Parts:
- AE1, BT1, J7, TP11, TP5, TP6, TP7, TP8, TP9: now not fitted; now left out of the parts list
- C1, C4: LCSC Part # (none) -> C723363
- C10, C11, C31, C8, C9: LCSC Part # (none) -> C60474
- C12, C21: LCSC Part # (none) -> C519560
- C13, C16, C17, C7: LCSC Part # (none) -> C7432767
- C18: LCSC Part # (none) -> C435397
- C19: LCSC Part # (none) -> C22374842
- C2, C32: LCSC Part # (none) -> C106861
- C20: LCSC Part # (none) -> C281756
- C3: LCSC Part # (none) -> C5137480
- C33: LCSC Part # (none) -> C723329
- C5, C6: LCSC Part # (none) -> C541383
- D1: LCSC Part # (none) -> C51933306
- FB1: LCSC Part # (none) -> C141722
- H2, JP1: now not fitted
- J5, J6: footprint Connector_PinHeader_2.54mm:PinHeader_1x20_P2.54mm_Vertical -> nrf54:Castellated_1x20_P2.54mm_Vertical; now not fitted; now left out of the parts list
- J8: footprint Connector_USB:USB_C_Receptacle_HRO_TYPE-C-31-M-12 -> PCM_ckl-connector:USB_C_Receptacle_HRO_TYPE-C-31-M-12; LCSC Part # C393939 -> C2681555
- J9: LCSC Part # (none) -> C88374
- L1: LCSC Part # (none) -> C394952
- L2: LCSC Part # C22471111 -> C5832372
- L3: LCSC Part # (none) -> C337946
- L4, L5: LCSC Part # (none) -> C3911055
- Q2: LCSC Part # C253528 -> C42412321
- R1, R8: LCSC Part # (none) -> C2906861
- R2: footprint Capacitor_SMD:C_0402_1005Metric -> Resistor_SMD:R_0402_1005Metric; LCSC Part # (none) -> C163830
- R9: LCSC Part # (none) -> C2906900
- SW1, SW2: LCSC Part # (none) -> C2888428
Other:
- moved on the sheet: C13

Commit message: Add schematic
Parts:
- AE1: value Antenna_Shield -> Antenna
- BT1: value Battery_Cell -> Battery
Other:
- note removed: "TODO: Changable to 3.3v"
- title: (none) -> nRF54L15 Discovery
- moved on the sheet: AE1, BT1, C1, C10, C11, C12, C13, C16, C17, C18, C19, C2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
